File: uniprog21.brd (EAGLE design)
At the start: 38 parts

Commit message: .
Parts:
- added D4, D5, D6, D7: КР580ВВ55, micro-intel:DIL40
- added X1: (no value), con-subd:M25HP
Connections:
- new net !IOWR: D4.36, D5.36
- new net P0: D4.4
- new net P1: D4.3
- new net P10: D4.20
- new net P11: D4.21
- new net P12: D4.22
- new net P13: D4.23
- new net P14: D4.24
- new net P15: D4.25
- new net P16: D4.14
- new net P17: D4.15
- new net P18: D4.16
- new net P19: D4.17
- new net P2: D4.2
- new net P20: D4.13
- new net P21: D4.12
- new net P22: D4.11
- new net P23: D4.10
- new net P24: D5.14
- new net P25: D5.15
- new net P26: D5.16
- new net P27: D5.17
- new net P28: D5.13
- new net P29: D5.12
- new net P3: D4.1
- new net P30: D5.11
- new net P31: D5.10
- new net P32: D5.18
- new net P33: D5.19
- new net P34: D5.20
- new net P35: D5.21
- new net P36: D5.22
- new net P37: D5.23
- new net P38: D5.24
- new net P39: D5.25
- new net P4: D4.40
- new net P40: D5.4
- new net P41: D5.3
- new net P42: D5.2
- new net P43: D5.1
- new net P44: D5.40
- new net P45: D5.39
- new net P46: D5.38
- new net P47: D5.37
- new net P48: D6.4
- new net P49: D6.3
- new net P5: D4.39
- new net P50: D6.2
- new net P51: D6.1
- new net P52: D6.40
- new net P53: D6.39
- new net P54: D6.38
- new net P55: D6.37
- new net P56: D6.18
- new net P57: D6.19
- new net P58: D6.20
- new net P59: D6.21
- new net P6: D4.38
- new net P60: D6.22
- new net P61: D6.23
- new net P62: D6.24
- new net P63: D6.25
- new net P68: D6.13
- new net P7: D4.37
- new net P8: D4.18
- new net P85: D7.23
- new net P9: D4.19
- new net RES: D4.35, D5.35
- new net XA0: D4.9, D5.9
- new net XA1: D4.8, D5.8
- new net XA6: D5.6
- new net XA7: D4.6
- net !IORD: now also D4.5, D5.5
- net +5V: now also D4.26, D5.26
- net D0: now also D4.34, D5.34, D6.34, D7.34
- net D1: now also D4.33, D5.33, D6.33, D7.33
- net D2: now also D4.32, D5.32, D6.32, D7.32
- net D3: now also D4.31, D5.31, D6.31, D7.31
- net D4: now also D4.30, D5.30, D6.30, D7.30
- net D5: now also D4.29, D5.29, D6.29, D7.29
- net D6: now also D4.28, D5.28, D6.28, D7.28
- net D7: now also D4.27, D5.27, D6.27, D7.27
- net GND: now also D4.7, D5.7, D6.7, D7.7
- net P64: now also D6.14
- net P65: now also D6.15
- net P66: now also D6.16
- net P67: now also D6.17
- net P69: now also D6.12
- net P70: now also D6.11
- net P71: now also D6.10
- net P72: now also D7.4
- net P73: now also D7.3
- net P74: now also D7.2
- net P75: now also D7.1
- net P76: now also D7.40
- net P77: now also D7.39
- net P78: now also D7.38
- net P79: now also D7.37
- net P80: now also D7.18
- net P81: now also D7.19
- net P82: now also D7.20
- net P83: now also D7.21
- net P84: now also D7.22
- net P86: now also D7.24
- net P87: now also D7.25
- net P88: now also D7.14
- net P89: now also D7.15
- net P90: now also D7.16
- net P91: now also D7.17
- net P92: now also D7.13
- net P93: now also D7.12
- net P94: now also D7.11
- net P95: now also D7.10
- net VCC: now also D6.26, D7.26

Commit message: .
Parts:
- removed D4, D5, D6, D7: КР580ВВ55, micro-intel:DIL40
- removed X1: (no value), con-subd:M25HP
- added C8: 47n, rcl:C0805
- added DD1: К555АП6, 74xx-eu:DIL20
- added DD2: К555КП11, 74xx-eu:DIL16
- added DD29: К555ИР23, 74xx-eu:DIL20
- added DD4, DD5, DD6, DD7: КР580ВВ55, micro-intel:DIL40
- added LPT: (no value), con-subd:M25HP
- added R68: 1k2, rcl:R0805
- renumbered D10 to DD10, D11 to DD11, D12 to DA12, D13 to DA13, D24 to DD24, D26 to DD26, D27 to DD27, D28 to DD28, D8 to DD8, D9 to DD9
Connections:
- new net !ADWR: DD1.19, DD29.11, LPT.14, R68.1
- new net !RDI: LPT.16
- new net !RSS: C8.1, DD24.11
- new net XA2: DD29.6
- new net XA4: DD29.12, DD7.6
- new net XA5: DD29.15, DD6.6
- new net XD0: DD1.2, DD29.3, LPT.2
- new net XD1: DD1.3, DD29.4, LPT.3
- new net XD2: DD1.4, DD29.7, LPT.4
- new net XD3: DD1.5, DD29.8, LPT.5
- new net XD4: DD1.6, DD29.13, LPT.6
- new net XD5: DD1.7, DD29.14, LPT.7
- new net XD6: DD1.8, DD29.17, LPT.8
- new net XD7: DD1.9, DD29.18, LPT.9
- new net XI0: DD2.4, LPT.13
- new net XI1: DD2.7, LPT.12
- new net XI2: DD2.9, LPT.10
- new net XI3: DD2.12, LPT.11
- new net XI4: DD2.1, LPT.1
- net !IORD: now also DD4.5, DD5.5, DD6.5, DD7.5; no longer D4.5, D5.5
- net !IOWR: now also DD4.36, DD5.36, DD6.36, DD7.36, LPT.17; no longer D4.36, D5.36
- net +5V: now also DD1.1, DD4.26, DD5.26, DD6.26, DD7.26, R68.2; no longer D4.26, D5.26
- net D0: now also DD1.18, DD2.2, DD4.34, DD5.34, DD6.34, DD7.34; no longer D4.34, D5.34, D6.34, D7.34
- net D1: now also DD1.17, DD2.5, DD4.33, DD5.33, DD6.33, DD7.33; no longer D4.33, D5.33, D6.33, D7.33
- net D2: now also DD1.16, DD2.11, DD4.32, DD5.32, DD6.32, DD7.32; no longer D4.32, D5.32, D6.32, D7.32
- net D3: now also DD1.15, DD2.14, DD4.31, DD5.31, DD6.31, DD7.31; no longer D4.31, D5.31, D6.31, D7.31
- net D4: now also DD1.14, DD2.3, DD4.30, DD5.30, DD6.30, DD7.30; no longer D4.30, D5.30, D6.30, D7.30
- net D5: now also DD1.13, DD2.6, DD4.29, DD5.29, DD6.29, DD7.29; no longer D4.29, D5.29, D6.29, D7.29
- net D6: now also DD1.12, DD2.10, DD4.28, DD5.28, DD6.28, DD7.28; no longer D4.28, D5.28, D6.28, D7.28
- net D7: now also DD1.11, DD2.13, DD4.27, DD5.27, DD6.27, DD7.27; no longer D4.27, D5.27, D6.27, D7.27
- net GND: now also C8.2, DD1.10, DD2.15, DD2.8, DD29.1, DD29.10, DD4.7, DD5.7, DD6.7, DD7.7, LPT.19, LPT.20, LPT.21, LPT.22, LPT.23, LPT.24, LPT.25; no longer D4.7, D5.7, D6.7, D7.7
- net P0: now also DD4.4; no longer D4.4
- net P1: now also DD4.3; no longer D4.3
- net P10: now also DD4.20; no longer D4.20
- net P11: now also DD4.21; no longer D4.21
- net P12: now also DD4.22; no longer D4.22
- net P13: now also DD4.23; no longer D4.23
- net P14: now also DD4.24; no longer D4.24
- net P15: now also DD4.25; no longer D4.25
- net P16: now also DD4.14; no longer D4.14
- net P17: now also DD4.15; no longer D4.15
- net P18: now also DD4.16; no longer D4.16
- net P19: now also DD4.17; no longer D4.17
- net P2: now also DD4.2; no longer D4.2
- net P20: now also DD4.13; no longer D4.13
- net P21: now also DD4.12; no longer D4.12
- net P22: now also DD4.11; no longer D4.11
- net P23: now also DD4.10; no longer D4.10
- net P24: now also DD5.14; no longer D5.14
- net P25: now also DD5.15; no longer D5.15
- net P26: now also DD5.16; no longer D5.16
- net P27: now also DD5.17; no longer D5.17
- net P28: now also DD5.13; no longer D5.13
- net P29: now also DD5.12; no longer D5.12
- net P3: now also DD4.1; no longer D4.1
- net P30: now also DD5.11; no longer D5.11
- net P31: now also DD5.10; no longer D5.10
- net P32: now also DD5.18; no longer D5.18
- net P33: now also DD5.19; no longer D5.19
- net P34: now also DD5.20; no longer D5.20
- net P35: now also DD5.21; no longer D5.21
- net P36: now also DD5.22; no longer D5.22
- net P37: now also DD5.23; no longer D5.23
- net P38: now also DD5.24; no longer D5.24
- net P39: now also DD5.25; no longer D5.25
- net P4: now also DD4.40; no longer D4.40
- net P40: now also DD5.4; no longer D5.4
- net P41: now also DD5.3; no longer D5.3
- net P42: now also DD5.2; no longer D5.2
- net P43: now also DD5.1; no longer D5.1
- net P44: now also DD5.40; no longer D5.40
- net P45: now also DD5.39; no longer D5.39
- net P46: now also DD5.38; no longer D5.38
- net P47: now also DD5.37; no longer D5.37
- net P48: now also DD6.4; no longer D6.4
- net P49: now also DD6.3; no longer D6.3
- net P5: now also DD4.39; no longer D4.39
- net P50: now also DD6.2; no longer D6.2
- net P51: now also DD6.1; no longer D6.1
- net P52: now also DD6.40; no longer D6.40
- net P53: now also DD6.39; no longer D6.39
- net P54: now also DD6.38; no longer D6.38
- net P55: now also DD6.37; no longer D6.37
- net P56: now also DD6.18; no longer D6.18
- net P57: now also DD6.19; no longer D6.19
- net P58: now also DD6.20; no longer D6.20
- net P59: now also DD6.21; no longer D6.21
- net P6: now also DD4.38; no longer D4.38
- net P60: now also DD6.22; no longer D6.22
- net P61: now also DD6.23; no longer D6.23
- net P62: now also DD6.24; no longer D6.24
- net P63: now also DD6.25; no longer D6.25
- net P64: now also DD6.14; no longer D6.14
- net P65: now also DD6.15; no longer D6.15
- net P66: now also DD6.16; no longer D6.16
- net P67: now also DD6.17; no longer D6.17
- net P68: now also DD6.13; no longer D6.13
- net P69: now also DD6.12; no longer D6.12
- net P7: now also DD4.37; no longer D4.37
- net P70: now also DD6.11; no longer D6.11
- net P71: now also DD6.10; no longer D6.10
- net P72: now also DD7.4; no longer D7.4
- net P73: now also DD7.3; no longer D7.3
- net P74: now also DD7.2; no longer D7.2
- net P75: now also DD7.1; no longer D7.1
- net P76: now also DD7.40; no longer D7.40
- net P77: now also DD7.39; no longer D7.39
- net P78: now also DD7.38; no longer D7.38
- net P79: now also DD7.37; no longer D7.37
- net P8: now also DD4.18; no longer D4.18
- net P80: now also DD7.18; no longer D7.18
- net P81: now also DD7.19; no longer D7.19
- net P82: now also DD7.20; no longer D7.20
- net P83: now also DD7.21; no longer D7.21
- net P84: now also DD7.22; no longer D7.22
- net P85: now also DD7.23; no longer D7.23
- net P86: now also DD7.24; no longer D7.24
- net P87: now also DD7.25; no longer D7.25
- net P88: now also DD7.14; no longer D7.14
- net P89: now also DD7.15; no longer D7.15
- net P9: now also DD4.19; no longer D4.19
- net P90: now also DD7.16; no longer D7.16
- net P91: now also DD7.17; no longer D7.17
- net P92: now also DD7.13; no longer D7.13
- net P93: now also DD7.12; no longer D7.12
- net P94: now also DD7.11; no longer D7.11
- net P95: now also DD7.10; no longer D7.10
- net RES: now also DD24.10, DD4.35, DD5.35, DD6.35, DD7.35; no longer D4.35, D5.35
- net VCC: now also DD1.20, DD2.16, DD29.20; no longer D6.26, D7.26
- net XA0: now also DD29.2, DD4.9, DD5.9, DD6.9, DD7.9; no longer D4.9, D5.9
- net XA1: now also DD29.5, DD4.8, DD5.8, DD6.8, DD7.8; no longer D4.8, D5.8
- net XA3: now also DD29.9
- net XA6: now also DD29.16, DD5.6; no longer D5.6
- net XA7: now also DD29.19, DD4.6; no longer D4.6

Commit message: .
Parts:
- added R65: 400, rcl:R0805
- added R67: 1k, rcl:R0805
- added VT1: 315, m_transistor:SOT23
- moved DD1 95.3 mm to (109.2, -120.7)
- moved DD2 54.6 mm to (20.3, -116.8)
- moved C8 38.9 mm to (17.8, -132.7), flipped to the bottom, turned to 270 degrees
- moved DD7 38.2 mm to (143.5, -109.9), turned to 270 degrees
- moved DD29 31.9 mm to (74.9, -122.6)
- moved DD5 20.4 mm to (52.1, -97.2)
- moved DD6 19.7 mm to (106.0, -97.2)
- moved DD4 17.7 mm to (14.6, -78.7), turned to 90 degrees
- moved LPT 8.28 mm to (26.0, -128.9)
Connections:
- new net N$8: R67.2, VT1.1
- net !IORD: now also R65.2, VT1.2
- net !RDI: now also R67.1
- net +5V: now also DD1.20, DD2.16, DD29.20, VT1.3
- net GND: now also R65.1
- net VCC: no longer DD1.20, DD2.16, DD29.20

Commit message: .
Parts:
- added DD15, DD16, DD17: К155ЛН3, 74xx-eu:DIL14
- added R10, R11: 470, rcl:R0805
- added R1A, R1B, R1C, R1D: 2k, rcl:R0805
- added VT2: 361g, m_transistor:SOT23
- added VT41: 315, m_transistor:SOT23
- VT1: value 315 -> 361g
- moved VT1 106.2 mm to (-17.8, -33.7), turned to 0 degrees
- moved DD24 55.5 mm to (106.0, -6.99)
- moved DD4 25.6 mm to (-3.17, -97.2), turned to 180 degrees
Connections:
- new net E1: R10.2, R11.2, VT1.2, VT2.2
- new net N$10: R1B.2, VT1.3
- new net N$11: R10.1, R1A.2, VT1.1
- new net N$12: DD17.12, R1C.1
- new net N$13: R1D.2, VT2.3
- new net N$14: R11.1, R1C.2, VT2.1
- new net N$9: DD16.4, R1A.1
- net !IORD: now also VT41.2; no longer VT1.2
- net +5V: now also VT41.3; no longer VT1.3
- net GND: now also DD15.7, DD16.7, DD17.7
- net N$8: now also VT41.1; no longer VT1.1
- net P0: now also DD16.3
- net P1: now also DD17.13
- net P8: now also DD15.1
- net P9: now also DD15.11
- net PA0: now also DD15.2, R1B.1
- net PA1: now also DD15.10, R1D.1
- net VCC: now also DD15.14, DD16.14, DD17.14

Commit message: b0
Parts:
- DD2: value К555КП11 -> К531КП11
Changed lines of the file:
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@@
 <element name="R68" library="rcl" package="R0805" value="1k2" x="3.81" y="-119.38" rot="MR0"/>
 <element name="DD1" library="74xx-eu" package="DIL20" value="К555АП6" x="109.22" y="-120.65"/>
-<element name="DD2" library="74xx-eu" package="DIL16" value="К555КП11" x="20.32" y="-116.84"/>
+<element name="DD2" library="74xx-eu" package="DIL16" value="К531КП11" x="20.32" y="-116.84"/>
 <element name="DD29" library="74xx-eu" package="DIL20" value="К555ИР23" x="74.93" y="-122.555" rot="R180"/>
 <element name="C8" library="rcl" package="C0805" value="47n" x="17.78" y="-132.715" rot="MR270"/>

Commit message: d1
Parts:
- added R1: 3k3, rcl:M0805
- added R38: 1k, rcl:M0805
- added R50: 510, rcl:M0805
- added R54: 100, rcl:M0805
- added VT29: КТ972, m_transistor:TO126V
- added VT33: КТ805, m_transistor:TO220FV
- added VT37: КТ973, m_transistor:TO126V
- added X2: (no value), Разъёмы штырьковые 2.54мм:2X20
- moved C1 265.5 mm to (278.1, -78.7), turned to 90 degrees
- moved DD26 260.0 mm to (276.9, -74.9), turned to 90 degrees
- moved C3 257.5 mm to (275.6, -73.7), turned to 270 degrees
- moved C2 250.8 mm to (276.9, -67.3), turned to 0 degrees
- moved DA13 202.2 mm to (264.8, -55.9)
- moved DD10 202.2 mm to (243.2, -57.1)
- moved DD9 202.2 mm to (243.2, -41.9)
- moved DA12 202.2 mm to (265.4, -43.8)
- moved DD11 202.2 mm to (217.8, -41.9)
- moved DD8 202.2 mm to (216.5, -58.4)
- moved R46 202.2 mm to (261.6, -36.2)
- moved R47 202.2 mm to (266.7, -36.2)
- moved DD7 101.2 mm to (238.8, -75.6), turned to 0 degrees
- moved C4 88.7 mm to (127.0, -50.8)
- moved DD27 88.7 mm to (129.5, -49.5)
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Connections:
- new net N$15: DA12.1, R1.1, R38.2
- new net N$16: R50.2, R54.2, VT29.1, VT33.3
- new net N$19: R46.2, R50.1, VT29.3, VT37.3
- net +27V: now also VT29.2, VT33.2
- net -5V: now also VT37.2
- net E1: now also R1.2, R54.1, VT33.1, VT37.1
- net GND: now also R38.1
- net P67: no longer DD8.5
- net P68: now also DD8.5
- net P84: no longer DD10.4
- net P85: now also DD10.4

Commit message: .
Parts:
- added C7: 390, rcl:C0805
- added DA1: КР574УД2А, ОУ:DIL08
- added R2, R3, R4, R5, R6, R7: (no value), rcl:M0805
- added R8, R9: 1k6, rcl:M0805
- added VT10, VT11, VT12, VT13, VT3, VT4, VT5, VT6, VT7, VT8, VT9: (no value), m_transistor:TO126V
Connections:
- new net N$17: VT3.3, VT4.3
- new net N$18: R3.1
- new net N$20: VT3.2, VT4.2, VT5.3, VT6.2, VT7.3
- new net N$22: VT11.3, VT5.2, VT6.3, VT7.2, VT8.3, VT9.3
- new net N$23: R4.1
- new net N$24: VT10.3, VT8.2, VT9.2
- new net N$26: R3.2, R5.2, R6.1
- new net N$27: R2.1, VT10.2, VT11.2
- new net N$28: R4.2, R6.2, R7.1
- new net N$32: R9.1, VT12.3
- new net N$33: C7.1, VT13.2
- new net N$34: R8.1, VT13.3
- new net N$36: C7.2, DA1.2, R2.2, R5.1, VT12.2
- new net V+: DA1.3
- new net V-: DA1.7
- net +14V: now also VT4.1, VT6.1, VT7.1, VT8.1
- net +5V: now also R8.2, R9.2
- net +7V: now also VT11.1
- net GND: now also R7.2, VT10.1, VT12.1, VT13.1, VT3.1, VT5.1, VT9.1

Commit message: .
Parts:
- removed C1, C2, C7: 390, rcl:C0805
- removed DA1: КР574УД2А, ОУ:DIL08
- removed DP1: 155РЕ3, ic-package:SOCKET-16
- removed DP10: i8748/9, ic-package:DIL40
- removed DP11: x8x5x, ic-package:DIL40
- removed DP2: 556РТ12-15, ic-package:SOCKET-18
- removed DP3: 556РТ4, ic-package:SOCKET-16
- removed DP4: 556РТ5-7,16, ic-package:DIL24-6
- removed DP5: 556РТ1, ic-package:DIL28-6
- removed DP6: 1556Хxx, ic-package:SOCKET-20
- removed DP7: 2x1000-2x8000, ic-package:DIL32
- removed DP8: 2x64-2x512, ic-package:DIL28-6
- removed DP9: 2716-2732, ic-package:DIL24-6
- removed LPT: (no value), con-subd:M25HP
- removed R1: 3k3, rcl:M0805
- removed R2, R3, R4, R5, R6, R7: (no value), rcl:M0805
- removed R38: 1k, rcl:M0805
- removed R46, R47: 270, rcl:M0805
- removed R50: 510, rcl:M0805
- removed R54: 100, rcl:M0805
- removed R8, R9: 1k6, rcl:M0805
- removed VT10, VT11, VT12, VT13, VT3, VT4, VT5, VT6, VT7, VT8, VT9: (no value), m_transistor:TO126V
- removed VT29: КТ972, m_transistor:TO126V
- removed VT33: КТ805, m_transistor:TO220FV
- removed VT37: КТ973, m_transistor:TO126V
- added C1N, C2N: 390, rcl:C0805
- added CX2, CX49: 100n, rcl:C0805
- added DP10U: i8748/9, ic-package:DIL40
- added DP11N: 556РТ5, ic-package:DIL24-6
- added DP11U/DP12N: x8x5x, ic-package:DIL40
- added DP1U/N: 155РЕ3, ic-package:SOCKET-16
- added DP2U/N: 556РТ12,13,14,15, ic-package:SOCKET-18
- added DP3U/N: 556РТ4,11, ic-package:SOCKET-16
- added DP4U/N(11): 556РТ5,6,7,16/6,7,16, ic-package:DIL24-6
- added DP5U/N: 556РТ1, ic-package:DIL28-6
- added DP6U/N: 1556Хxx, ic-package:SOCKET-20
- added DP7U/DP8N: 2x1000-2x8000, ic-package:DIL32
- added DP8U/DP9N: 2x64-2x512, ic-package:DIL28-6
- added DP9U/DP10N: 2716-2732, ic-package:DIL24-6
- added LPT26PINS: (no value), Разъёмы штырьковые 2.54мм:2X13
- added LPTDB25_: (no value), con-subd:M25HP
- added R1/R87N, R92N: 3k3, rcl:M0805
- added R38/R88N, R93N: 1k, rcl:M0805
- added R46/R89N, R94N: 270, rcl:M0805
- added R50/R90N, R95N: 510, rcl:M0805
- added R54/R91N, R96N: 100, rcl:M0805
- added VT29N, VT30N: КТ972, m_transistor:TO126V
- added VT33N, VT34N: КТ805, m_transistor:TO220FV
- added VT37N, VT38N: КТ973, m_transistor:TO126V
- added X1: (no value), Разъёмы штырьковые 2.54мм:2X20
- moved C3 303.1 mm to (-21.6, -133.3)
- moved DD26 301.4 mm to (-19.1, -132.1)
- moved DD29 273.2 mm to (15.9, 144.1), turned to 0 degrees
- moved VT41 261.9 mm to (71.8, 114.9), turned to 90 degrees
- moved R65 258.3 mm to (64.1, 114.9), turned to 180 degrees
- moved DD1 256.4 mm to (15.9, 118.1)
- moved R67 254.2 mm to (66.0, 112.4), turned to 90 degrees
- moved DD9 251.8 mm to (13.3, -144.8), turned to 90 degrees
- moved DD2 247.7 mm to (13.3, 130.8)
- moved C8 245.7 mm to (57.1, 109.9), turned to 90 degrees
- moved DD7 229.6 mm to (13.3, -119.4), turned to 90 degrees
- moved DD10 229.3 mm to (15.9, -87.0)
- moved DD11 216.9 mm to (13.3, -114.3), turned to 90 degrees
- moved X2 194.0 mm to (54.6, 31.1), turned to 180 degrees
- moved DD8 191.2 mm to (33.7, -114.3), turned to 90 degrees
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Connections:
- removed net N$17: VT3.3, VT4.3
- removed net N$18: R3.1
- removed net N$2: C2.1, DD26.6
- removed net N$27: R2.1, VT10.2, VT11.2
- removed net N$28: R4.2, R6.2, R7.1
- removed net N$32: R9.1, VT12.3
- removed net N$33: C7.1, VT13.2
- removed net N$34: R8.1, VT13.3
- removed net N$36: C7.2, DA1.2, R2.2, R5.1, VT12.2
- removed net N$7: DA12.6, R47.1
- removed net V+: DA1.3
- removed net V-: DA1.7
- new net N$21: DD10.14, DD11.14
- new net N$25: R95N.2, R96N.2, VT30N.1, VT34N.3
- net !ADWR: now also LPT26PINS.2; no longer LPT.14
- net !EN1: now also C1N.2; no longer C1.2
- net !EN2: now also C2N.2; no longer C2.2
- net !EN3: now also DD27.12; no longer DD26.12
- net !IOWR: now also LPT26PINS.8; no longer LPT.17
- net !RDI: now also LPT26PINS.6; no longer LPT.16
- net +14V: no longer DD10.14, DD11.14, VT4.1, VT6.1, VT7.1, VT8.1
- net +27V: now also CX2.1, CX49.1, VT29N.2, VT30N.2, VT33N.2, VT34N.2; no longer VT29.2, VT33.2
- net +5V: now also DD26.14, DP11U/DP12N.9; no longer DP11.9, R8.2, R9.2
- net +7V: no longer DD10.1, DD11.1, VT11.1
- net -5V: now also CX2.2, CX49.2, VT37N.2, VT38N.2; no longer VT37.2
- net BQ1: now also DP11U/DP12N.19; no longer DP11.19
- net BQ2: now also DP11U/DP12N.18; no longer DP11.18
- net E1: now also R1/R87N.2, R54/R91N.1, VT33N.1, VT37N.1; no longer R1.2, R54.1, VT33.1, VT37.1
- net E2: now also DP11U/DP12N.40, DP5U/N.19, DP6U/N.11, R92N.2, R96N.1, VT34N.1, VT38N.1; no longer DP11.40, DP5.19, DP6.11
- net E3: now also DP11U/DP12N.30; no longer DP11.30
- net E4: now also DP11U/DP12N.31, DP5U/N.28, DP6U/N.20; no longer DP11.31, DP5.28, DP6.20
- net GND: now also DP11U/DP12N.20, DP11U/DP12N.29, DP5U/N.14, DP6U/N.10, LPT26PINS.10, LPT26PINS.12, LPT26PINS.14, LPT26PINS.16, LPT26PINS.18, LPT26PINS.20, LPT26PINS.22, LPT26PINS.24, LPT26PINS.26, R38/R88N.1, R93N.1; no longer DP11.20, DP11.29, DP5.14, DP6.10, LPT.19, LPT.20, LPT.21, LPT.22, LPT.23, LPT.24, LPT.25, R38.1, R7.2, VT10.1, VT12.1, VT13.1, VT3.1, VT5.1, VT9.1
- net N$1: now also C1N.1; no longer C1.1
- net N$15: now also R1/R87N.1, R38/R88N.2; no longer R1.1, R38.2
- net N$16: now also R50/R90N.2, R54/R91N.2, VT29N.1, VT33N.3; no longer R50.2, R54.2, VT29.1, VT33.3
- net N$19: now also R46/R89N.2, R50/R90N.1, VT29N.3, VT37N.3; no longer R46.2, R50.1, VT29.3, VT37.3
- net N$20: now also DD10.1, DD11.1; no longer VT3.2, VT4.2, VT5.3, VT6.2, VT7.3
- net N$22: now also C2N.1, DD26.6; no longer VT11.3, VT5.2, VT6.3, VT7.2, VT8.3, VT9.3
- net N$23: now also DA12.6, R94N.1; no longer R4.1
- net N$24: now also DA12.5, R92N.1, R93N.2; no longer VT10.3, VT8.2, VT9.2
- net N$26: now also R94N.2, R95N.1, VT30N.3, VT38N.3; no longer R3.2, R5.2, R6.1
- net N$3: now also DD27.10; no longer DD26.10
- net N$6: now also R46/R89N.1; no longer R46.1
- net P86: now also DD27.11; no longer DD26.11
- net P87: now also DD27.13; no longer DD26.13
- net PA0: now also DP11U/DP12N.1; no longer DP11.1
- net PA1: now also DP11U/DP12N.2; no longer DP11.2
- net PA10: now also DP11U/DP12N.23, DP5U/N.25; no longer DP11.23, DP5.25
- net PA11: now also DP11U/DP12N.24, DP5U/N.24; no longer DP11.24, DP5.24
- net PA12: now also DP11U/DP12N.25, DP5U/N.23; no longer DP11.25, DP5.23
- net PA13: now also DP10U.36, DP11U/DP12N.26, DP5U/N.22; no longer DP11.26, DP5.22
- net PA14: now also DP10U.37, DP11U/DP12N.27, DP5U/N.21; no longer DP11.27, DP5.21
- net PA15: now also DP10U.38, DP11U/DP12N.28, DP5U/N.20; no longer DP10.38, DP11.28, DP5.20
- net PA16: now also DP11U/DP12N.10, DP11U/DP12N.14; no longer DP11.10, DP11.14
- net PA17: now also DP11U/DP12N.13; no longer DP11.13
- net PA18: now also DP11U/DP12N.16; no longer DP11.16
- net PA19: now also DP11U/DP12N.17; no longer DP11.17
- net PA2: now also DP11U/DP12N.3; no longer DP11.3
- net PA3: now also DP11U/DP12N.4; no longer DP11.4
- net PA4: now also DP11U/DP12N.5; no longer DP11.5
- net PA5: now also DP11U/DP12N.6; no longer DP11.6
- net PA6: now also DP11U/DP12N.7; no longer DP11.7
- net PA7: now also DP11U/DP12N.8; no longer DP11.8
- net PA8: now also DP11U/DP12N.21, DP5U/N.27; no longer DP11.21, DP5.27
- net PA9: now also DP11U/DP12N.22, DP5U/N.26; no longer DP11.22, DP5.26
- net PD0: now also DP11U/DP12N.39, DP5U/N.18, DP6U/N.19; no longer DP11.39, DP5.18, DP6.19
- net PD1: now also DP11U/DP12N.38, DP5U/N.17, DP6U/N.18; no longer DP11.38, DP5.17, DP6.18
- net PD2: now also DP11U/DP12N.37, DP5U/N.16, DP6U/N.17; no longer DP11.37, DP5.16, DP6.17
- net PD3: now also DP11U/DP12N.36, DP5U/N.15, DP6U/N.16; no longer DP11.36, DP5.15, DP6.16
- net PD4: now also DP11U/DP12N.35, DP6U/N.15; no longer DP11.35, DP6.15
- net PD5: now also DP11U/DP12N.34, DP6U/N.14; no longer DP11.34, DP6.14
- net PD6: now also DP11U/DP12N.33, DP6U/N.13; no longer DP11.33, DP6.13
- net PD7: now also DP11U/DP12N.32, DP6U/N.12; no longer DP11.32, DP6.12
- net VCC: no longer DD26.14
- net XD0: now also LPT26PINS.3; no longer LPT.2
- net XD1: now also LPT26PINS.5; no longer LPT.3
- net XD2: now also LPT26PINS.7; no longer LPT.4
- net XD3: now also LPT26PINS.9; no longer LPT.5
- net XD4: now also LPT26PINS.11; no longer LPT.6
- net XD5: now also LPT26PINS.13; no longer LPT.7
- net XD6: now also LPT26PINS.15; no longer LPT.8
- net XD7: now also LPT26PINS.17; no longer LPT.9
- net XI0: now also LPT26PINS.25; no longer LPT.13
- net XI1: now also LPT26PINS.23; no longer LPT.12
- net XI2: now also LPT26PINS.19; no longer LPT.10
- net XI3: now also LPT26PINS.21; no longer LPT.11
- net XI4: now also LPT26PINS.1; no longer LPT.1
Routing:
- net GND: track 0.00 -> 115.3 mm
- net +5V: track 0.00 -> 101.5 mm
- net XD7: track 0.00 -> 71.0 mm
- net D7: track 0.00 -> 65.2 mm
- net D5: track 0.00 -> 65.2 mm
- net D6: track 0.00 -> 65.2 mm
- net D4: track 0.00 -> 65.2 mm
- net D3: track 0.00 -> 64.8 mm
- net XA1: track 0.00 -> 64.1 mm
- net RES: track 0.00 -> 64.1 mm
- net !IOWR: track 0.00 -> 64.1 mm
- net D1: track 0.00 -> 64.1 mm
- net D0: track 0.00 -> 64.1 mm
- net !IORD: track 0.00 -> 64.1 mm
- net XA0: track 0.00 -> 63.8 mm
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