File: uniprog21.brd (EAGLE design)
At the start: 82 parts

Commit message: .
Parts:
- removed C3, C4: 390, rcl:C0805
- added C3N, C4N: 390, rcl:C0805
- added R100N, R105N: 510, rcl:M0805
- added R101, R106N: 100, rcl:M0805
- added R102N, R97N: 3k3, rcl:M0805
- added R103N, R98N: 1k, rcl:M0805
- added R104N, R99N: 270, rcl:M0805
- added VT31N, VT32N: КТ972, m_transistor:TO126V
- added VT35N, VT36N: КТ805, m_transistor:TO220FV
- added VT39N, VT40N: КТ973, m_transistor:TO126V
- moved DD27 96.7 mm to (123.2, -146.1), turned to 270 degrees
- moved DD24 11.4 mm to (106.0, -56.5), turned to 270 degrees
Connections:
- removed net N$20: DD10.1, DD11.1
- removed net N$21: DD10.14, DD11.14
- removed net N$3: C3.1, DD27.10
- removed net N$4: C4.1, DD27.2
- new net N$17: DA13.1, R97N.1, R98N.2
- new net N$18: R100N.2, R101.2, VT31N.1, VT35N.3
- new net N$2: C3N.1, DD27.10
- new net N$27: R100N.1, R99N.2, VT31N.3, VT39N.3
- new net N$28: C4N.1, DD27.2
- new net N$29: DA13.6, R104N.1
- new net N$30: DA13.5, R102N.1, R103N.2
- new net N$31: R105N.2, R106N.2, VT32N.1, VT36N.3
- new net N$32: R104N.2, R105N.1, VT32N.3, VT40N.3
- new net N$7: DA13.8, R99N.1
- net !EN3: now also C3N.2, DA13.2; no longer C3.2
- net !EN4: now also C4N.2, DA13.4; no longer C4.2
- net +14V: now also DD10.14, DD11.14
- net +27V: now also VT31N.2, VT32N.2, VT35N.2, VT36N.2
- net +5V: now also DD27.14
- net +7V: now also DD10.1, DD11.1
- net -5V: now also VT39N.2, VT40N.2
- net E3: now also R101.1, R97N.2, VT35N.1, VT39N.1
- net E4: now also R102N.2, R106N.1, VT36N.1, VT40N.1
- net GND: now also R103N.1, R98N.1
- net VCC: no longer DD27.14
Routing:
- net GND: track 115.3 -> 106.6 mm
