File: uniprog21.brd (EAGLE design)
At the start: 98 parts

Commit message: .
Parts:
- removed R10, R11: 470, rcl:R0805
- removed R1A, R1B, R1C, R1D: 2k, rcl:R0805
- removed R5A, R5B, R5C, R5D, R5E, R5F, R5G, R5H: 1k, rcl:M0805
- added JP1: (no value), Разъёмы штырьковые 2.54мм:1X06
- added JP2: (no value), Разъёмы штырьковые 2.54мм:1X04
- added JP3: (no value), Разъёмы штырьковые 2.54мм:1X11
- added JP5: (no value), Разъёмы штырьковые 2.54мм:1X05
- added R83(R62U2.1), R84(R5U2.1), R85(R6U2.1), R86(R8U2.1): 1k, resistor-sil:SIL10
- added RN1: НР-1-1-1-8 470 5%, resistor-dil:DIL16
- added RN10: НР-1-1-1-8 2k, resistor-dil:DIL16
- added VD1, VD10, VD11, VD12, VD13, VD14, VD15, VD16, VD2, VD3, VD4, VD5, VD6, VD7, VD8, VD9: КД522, diode:DO35-7
- VT1, VT2: value 361g -> КТ361Г; device m_transistor:SOT23 -> m_transistor:TO92
- moved DD27 154.9 mm to (-24.8, -100.3), turned to 90 degrees
- moved DD10 79.9 mm to (-61.6, -106.7), turned to 90 degrees
- moved VT2 66.6 mm to (-56.5, 95.9), flipped to the top
- moved VT1 45.5 mm to (-63.5, 95.9), flipped to the top
- moved DD9 43.9 mm to (-30.5, -142.2)
- moved DD15 39.1 mm to (-40.0, 41.3)
- moved DD17 30.8 mm to (-33.0, 70.5)
- moved DD28 20.7 mm to (-59.1, 11.4)
- moved C1N 18.5 mm to (-30.5, -123.8)
- moved VT31N 17.1 mm to (191.1, -88.9)
- moved VT32N 16.2 mm to (201.9, -86.4), turned to 270 degrees
- moved DD26 15.4 mm to (-28.6, -120.0)
- moved VT36N 14.8 mm to (189.9, -80.6)
- moved DD16 14.1 mm to (-50.2, 57.8)
- moved VT34N 9.53 mm to (168.9, -133.3)
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Connections:
- new net N$20: VD9.A
- new net N$21: R85(R6U2.1).3, VD10.C
- new net N$3: R85(R6U2.1).2, VD9.C
- new net N$33: R85(R6U2.1).4, VD11.C
- new net N$34: R85(R6U2.1).5, VD12.C
- new net N$35: R85(R6U2.1).6, VD13.C
- new net N$36: R85(R6U2.1).7, VD14.C
- new net N$37: R85(R6U2.1).8, VD15.C
- new net N$38: R85(R6U2.1).9, VD16.C
- new net N$4: VD10.A
- net !IOWR: now also JP1.2
- net +5V: now also R83(R62U2.1).1, R84(R5U2.1).1; no longer R5A.2, R5B.2, R5C.2, R5D.2, R5E.2, R5F.2, R5G.2, R5H.2
- net E1: now also RN1.14, RN1.16, VT1.1, VT2.1; no longer R10.2, R11.2, VT1.2, VT2.2
- net N$10: now also RN1.15, VT1.2; no longer R1B.2, VT1.3
- net N$11: now also RN1.1, RN10.16, VT1.3; no longer R10.1, R1A.2, VT1.1
- net N$12: now also RN10.2; no longer R1C.1
- net N$13: now also RN1.13, VT2.2; no longer R1D.2, VT2.3
- net N$14: now also RN1.3, RN10.15, VT2.3; no longer R11.1, R1C.2, VT2.1
- net N$9: now also RN10.1; no longer R1A.1
- net P72: now also JP2.4
- net P73: now also JP2.3
- net P74: now also JP2.2
- net P75: now also JP2.1
- net P76: now also JP1.6
- net P77: now also JP1.5
- net P78: now also JP1.4
- net P79: now also JP1.3
- net P80: now also JP3.9
- net P81: now also JP3.10
- net P82: now also JP3.11
- net P83: now also JP5.1
- net P84: now also JP5.2
- net P85: now also JP5.3
- net P86: now also JP5.4
- net P87: now also JP5.5
- net P88: now also JP3.5
- net P89: now also JP3.6
- net P90: now also JP3.7
- net P91: now also JP3.8
- net P92: now also JP3.4
- net P93: now also JP3.3
- net P94: now also JP3.2
- net P95: now also JP3.1
- net PA0: now also RN1.2; no longer R1B.1
- net PA1: now also RN1.4; no longer R1D.1
- net PD10: now also R84(R5U2.1).4; no longer R5C.1
- net PD11: now also R84(R5U2.1).5, R84(R5U2.1).6; no longer R5D.1, R5E.1
- net PD13: now also R84(R5U2.1).7; no longer R5F.1
- net PD14: now also R84(R5U2.1).8; no longer R5G.1
- net PD15: now also R84(R5U2.1).9; no longer R5H.1
- net PD8: now also R84(R5U2.1).2; no longer R5A.1
- net PD9: now also R84(R5U2.1).3; no longer R5B.1
- net RES: now also JP1.1
Routing:
- net P75: track 4.58 -> 46.6 mm
- net P74: track 4.58 -> 46.6 mm
- net P73: track 4.58 -> 46.6 mm
- net E1: track 0.00 -> 18.9 mm
- net N$14: track 0.00 -> 18.1 mm
- net N$11: track 0.00 -> 16.4 mm
- net N$25: track 5.02 -> 17.2 mm
- net +27V: track 16.5 -> 23.6 mm
- net N$26: track 12.1 -> 16.9 mm
- net N$10: track 0.00 -> 3.70 mm
- net N$13: track 0.00 -> 3.17 mm
- net E2: track 12.0 -> 14.1 mm
- net RES: track 64.1 -> 65.4 mm
- net GND: track 106.6 -> 107.9 mm
- net !IOWR: track 64.1 -> 65.4 mm
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
Commit message: .
Parts:
- removed DD15, DD16: К155ЛН3, 74xx-eu:DIL14
- added (DD15.1)DD15, (DD16.1)DD14, D-0, D-1, D-2: К155ЛН3, 74xx-eu:DIL14
- added D1, D10, D11, D2, D3, D4, D5, D6, D7, D8, D9: Д310, diode:DO15-12
- added R1, R10, R11, R12, R19, R2, R20, R21, R3: 2k, rcl:R0805
- added R13, R14, R15, R16, R17, R18, R22, R23, R24, R25, R26, R27, R4, R5, R6, R7, R8, R9: 470, rcl:R0805
- added VT10, VT11, VT3, VT4, VT5, VT6, VT7, VT8, VT9: КТ361Г, m_transistor:TO92
- R1/R87N, R100N, R101, R102N, R103N, R104N, R105N, R106N, R38/R88N, R46/R89N, R50/R90N, R54/R91N, R92N, R93N, R94N, R95N, R96N, R97N, R98N, R99N: device rcl:M0805 -> rcl:R0805
- moved C2N 328.3 mm to (-200.0, -85.7)
- moved C3N 328.3 mm to (-120.0, -99.7)
- moved C4N 328.3 mm to (-113.7, -99.7)
- moved R100N 328.3 mm to (-102.2, -85.1)
- moved R101 328.3 mm to (-134.0, -93.3)
- moved R104N 328.3 mm to (-98.4, -93.3)
- moved R105N 328.3 mm to (-134.0, -99.7)
- moved R96N 328.3 mm to (-163.8, -111.1)
- moved R99N 328.3 mm to (-113.7, -85.1)
- moved VT32N 328.3 mm to (-125.7, -66.7)
- moved VT39N 328.3 mm to (-102.2, -73.7)
- moved CX2 328.3 mm to (-194.3, -95.9)
- moved CX49 328.3 mm to (-175.9, -51.4)
- moved DA12 328.3 mm to (-194.3, -94.6)
- moved DA13 328.3 mm to (-174.6, -51.4)
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- renumbered JP1 to P_DAC4, JP2 to P_DAC1, JP3 to P_DAC2, JP5 to P_DAC3
Connections:
- new net N$39: D1.A, RN1.2
- new net N$40: D2.A, RN1.4
- new net N$41: R1.2, R4.1, VT3.3
- new net N$42: D6.A, VT3.2
- new net N$43: D6.C, R5.2
- new net N$44: D-0.2, R1.1
- new net N$45: R2.2, R6.1, VT4.3
- new net N$46: D3.A, VT4.2
- new net N$47: D-0.12, R5.1
- new net N$48: R3.2, R8.1, VT5.3
- new net N$49: D4.A, VT5.2
- new net N$50: D-0.8, R9.1
- new net N$51: D-0.6, R3.1
- new net N$52: D-0.4, R2.1
- new net N$53: D4.C, R9.2
- new net N$54: D3.C, R7.2
- new net N$55: D-0.10, R7.1
- new net N$56: R10.2, R13.1, VT7.3
- new net N$57: D5.A, VT7.2
- new net N$58: D-1.2, R10.1
- new net N$59: R11.2, R15.1, VT8.3
- new net N$60: D7.A, VT8.2
- new net N$61: R12.2, R17.1, VT9.3
- new net N$62: D8.A, VT9.2
- new net N$63: D-1.6, R12.1
- new net N$64: D-1.4, R11.1
- new net N$65: D5.C, R14.2
- new net N$66: D-1.12, R14.1
- new net N$67: D-1.8, R18.1
- new net N$68: D8.C, R18.2
- new net N$69: D7.C, R16.2
- new net N$70: D-1.10, R16.1
- new net N$71: R19.2, R22.1, VT6.3
- new net N$72: D9.A, VT6.2
- new net N$73: D-2.2, R19.1
- new net N$74: R20.2, R24.1, VT10.3
- new net N$75: D10.A, VT10.2
- new net N$76: R21.2, R26.1, VT11.3
- new net N$77: D11.A, VT11.2
- new net N$78: D-2.6, R21.1
- new net N$79: D-2.4, R20.1
- new net N$80: D9.C, R23.2
- new net N$81: D-2.12, R23.1
- new net N$82: D-2.8, R27.1
- new net N$83: D11.C, R27.2
- new net N$84: D10.C, R25.2
- new net N$85: D-2.10, R25.1
- net E1: now also R13.2, R15.2, R17.2, R22.2, R24.2, R26.2, R4.2, R6.2, R8.2, VT10.1, VT11.1, VT3.1, VT4.1, VT5.1, VT6.1, VT7.1, VT8.1, VT9.1
- net GND: now also (DD15.1)DD15.7, (DD16.1)DD14.7, D-0.7, D-1.7, D-2.7; no longer DD15.7, DD16.7
- net N$9: now also (DD16.1)DD14.6; no longer DD16.4
- net P0: now also (DD16.1)DD14.5; no longer DD16.3
- net P8: now also (DD15.1)DD15.1; no longer DD15.1
- net P9: now also (DD15.1)DD15.11; no longer DD15.11
- net PA0: now also (DD15.1)DD15.2, D1.C; no longer DD15.2, RN1.2
- net PA1: now also (DD15.1)DD15.10, D2.C; no longer DD15.10, RN1.4
- net VCC: now also (DD15.1)DD15.14, (DD16.1)DD14.14, D-0.14, D-1.14, D-2.14; no longer DD15.14, DD16.14
Routing:
- net E1: track 18.9 -> 83.7 mm
- net N$44: track 0.00 -> 11.5 mm
- net N$52: track 0.00 -> 11.3 mm
- net N$51: track 0.00 -> 11.3 mm
- net N$55: track 0.00 -> 7.52 mm
- net N$47: track 0.00 -> 7.00 mm
- net N$62: track 0.00 -> 6.66 mm
- net N$60: track 0.00 -> 6.40 mm
- net N$49: track 0.00 -> 6.40 mm
- net N$42: track 0.00 -> 6.40 mm
- net N$57: track 0.00 -> 6.40 mm
- net N$46: track 0.00 -> 6.40 mm
- net N$10: track 3.70 -> 0.00 mm
- net N$13: track 3.17 -> 0.00 mm
- net N$50: track 0.00 -> 2.86 mm
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