File: uniprog21.sch (EAGLE design)
At the start: 38 parts

Commit message: .
Parts:
- added D4, D5, D6, D7: КР580ВВ55, micro-intel:82C55A
- added X1: (no value), con-subd:M25HP
Connections:
- new net !IOWR: D4.WR, D5.WR
- new net P0: D4.PA0
- new net P1: D4.PA1
- new net P10: D4.PB2
- new net P11: D4.PB3
- new net P12: D4.PB4
- new net P13: D4.PB5
- new net P14: D4.PB6
- new net P15: D4.PB7
- new net P16: D4.PC0
- new net P17: D4.PC1
- new net P18: D4.PC2
- new net P19: D4.PC3
- new net P2: D4.PA2
- new net P20: D4.PC4
- new net P21: D4.PC5
- new net P22: D4.PC6
- new net P23: D4.PC7
- new net P24: D5.PC0
- new net P25: D5.PC1
- new net P26: D5.PC2
- new net P27: D5.PC3
- new net P28: D5.PC4
- new net P29: D5.PC5
- new net P3: D4.PA3
- new net P30: D5.PC6
- new net P31: D5.PC7
- new net P32: D5.PB0
- new net P33: D5.PB1
- new net P34: D5.PB2
- new net P35: D5.PB3
- new net P36: D5.PB4
- new net P37: D5.PB5
- new net P38: D5.PB6
- new net P39: D5.PB7
- new net P4: D4.PA4
- new net P40: D5.PA0
- new net P41: D5.PA1
- new net P42: D5.PA2
- new net P43: D5.PA3
- new net P44: D5.PA4
- new net P45: D5.PA5
- new net P46: D5.PA6
- new net P47: D5.PA7
- new net P48: D6.PA0
- new net P49: D6.PA1
- new net P5: D4.PA5
- new net P50: D6.PA2
- new net P51: D6.PA3
- new net P52: D6.PA4
- new net P53: D6.PA5
- new net P54: D6.PA6
- new net P55: D6.PA7
- new net P56: D6.PB0
- new net P57: D6.PB1
- new net P58: D6.PB2
- new net P59: D6.PB3
- new net P6: D4.PA6
- new net P60: D6.PB4
- new net P61: D6.PB5
- new net P62: D6.PB6
- new net P63: D6.PB7
- new net P68: D6.PC4
- new net P7: D4.PA7
- new net P8: D4.PB0
- new net P85: D7.PB5
- new net P9: D4.PB1
- new net RES: D4.RESET, D5.RESET
- new net XA0: D4.A0, D5.A0
- new net XA1: D4.A1, D5.A1
- new net XA6: D5.CS
- new net XA7: D4.CS
- net !IORD: now also D4.RD, D5.RD
- net +5V: now also D4.VCC, D5.VCC
- net D0: now also D4.D0, D5.D0, D6.D0, D7.D0
- net D1: now also D4.D1, D5.D1, D6.D1, D7.D1
- net D2: now also D4.D2, D5.D2, D6.D2, D7.D2
- net D3: now also D4.D3, D5.D3, D6.D3, D7.D3
- net D4: now also D4.D4, D5.D4, D6.D4, D7.D4
- net D5: now also D4.D5, D5.D5, D6.D5, D7.D5
- net D6: now also D4.D6, D5.D6, D6.D6, D7.D6
- net D7: now also D4.D7, D5.D7, D6.D7, D7.D7
- net GND: now also D4.GND, D5.GND
- net P64: now also D6.PC0
- net P65: now also D6.PC1
- net P66: now also D6.PC2
- net P67: now also D6.PC3
- net P69: now also D6.PC5
- net P70: now also D6.PC6
- net P71: now also D6.PC7
- net P72: now also D7.PA0
- net P73: now also D7.PA1
- net P74: now also D7.PA2
- net P75: now also D7.PA3
- net P76: now also D7.PA4
- net P77: now also D7.PA5
- net P78: now also D7.PA6
- net P79: now also D7.PA7
- net P80: now also D7.PB0
- net P81: now also D7.PB1
- net P82: now also D7.PB2
- net P83: now also D7.PB3
- net P84: now also D7.PB4
- net P86: now also D7.PB6
- net P87: now also D7.PB7
- net P88: now also D7.PC0
- net P89: now also D7.PC1
- net P90: now also D7.PC2
- net P91: now also D7.PC3
- net P92: now also D7.PC4
- net P93: now also D7.PC5
- net P94: now also D7.PC6
- net P95: now also D7.PC7

Commit message: .
Parts:
- removed D24: 555ЛН1, 74xx-eu:74LS04N
- removed D6, D7: КР580ВВ55, micro-intel:82C55A
- removed X1: (no value), con-subd:M25HP
- added C8: 47n, rcl:C-EUC0805
- added DD1: К555АП6, 74xx-eu:74LS245N
- added DD2: К555КП11, 74xx-eu:74S257N
- added DD24: 555ЛН1, 74xx-eu:74LS04N
- added DD29: К555ИР23, 74xx-eu:74LS374N
- added DD6, DD7: КР580ВВ55, micro-intel:82C55A
- added LPT: (no value), con-subd:M25HP
- added R68: 1k2, rcl:R-EU_R0805
- renumbered D10 to DD10, D11 to DD11, D12 to DA12, D13 to DA13, D26 to DD26, D27 to DD27, D28 to DD28, D4 to DD4, D5 to DD5, D8 to DD8, D9 to DD9
Connections:
- new net !ADWR: DD1A.G, DD29A.CLK, LPT.14, R68.1
- new net !RDI: LPT.16
- new net !RSS: C8.1, DD24E.I
- new net XA2: DD29A.3Q
- new net XA4: DD29A.5Q, DD7.CS
- new net XA5: DD29A.6Q, DD6.CS
- new net XD0: DD1A.A1, DD29A.1D, LPT.2
- new net XD1: DD1A.A2, DD29A.2D, LPT.3
- new net XD2: DD1A.A3, DD29A.3D, LPT.4
- new net XD3: DD1A.A4, DD29A.4D, LPT.5
- new net XD4: DD1A.A5, DD29A.5D, LPT.6
- new net XD5: DD1A.A6, DD29A.6D, LPT.7
- new net XD6: DD1A.A7, DD29A.7D, LPT.8
- new net XD7: DD1A.A8, DD29A.8D, LPT.9
- new net XI0: DD2A.1Y, LPT.13
- new net XI1: DD2A.2Y, LPT.12
- new net XI2: DD2A.3Y, LPT.10
- new net XI3: DD2A.4Y, LPT.11
- new net XI4: DD2A.!A!/B, LPT.1
- net !IORD: now also DD6.RD, DD7.RD
- net !IOWR: now also DD6.WR, DD7.WR, LPT.17
- net +5V: now also DD1A.DIR, DD6.VCC, DD7.VCC, R68.2
- net D0: now also DD1A.B1, DD2A.1A, DD6.D0, DD7.D0; no longer D6.D0, D7.D0
- net D1: now also DD1A.B2, DD2A.2A, DD6.D1, DD7.D1; no longer D6.D1, D7.D1
- net D2: now also DD1A.B3, DD2A.3A, DD6.D2, DD7.D2; no longer D6.D2, D7.D2
- net D3: now also DD1A.B4, DD2A.4A, DD6.D3, DD7.D3; no longer D6.D3, D7.D3
- net D4: now also DD1A.B5, DD2A.1B, DD6.D4, DD7.D4; no longer D6.D4, D7.D4
- net D5: now also DD1A.B6, DD2A.2B, DD6.D5, DD7.D5; no longer D6.D5, D7.D5
- net D6: now also DD1A.B7, DD2A.3B, DD6.D6, DD7.D6; no longer D6.D6, D7.D6
- net D7: now also DD1A.B8, DD2A.4B, DD6.D7, DD7.D7; no longer D6.D7, D7.D7
- net GND: now also C8.2, DD29A.OC, DD2A.G, DD6.GND, DD7.GND, LPT.19, LPT.20, LPT.21, LPT.22, LPT.23, LPT.24, LPT.25
- net N$5: now also DD24D.O; no longer D24D.O
- net P48: now also DD6.PA0; no longer D6.PA0
- net P49: now also DD6.PA1; no longer D6.PA1
- net P50: now also DD6.PA2; no longer D6.PA2
- net P51: now also DD6.PA3; no longer D6.PA3
- net P52: now also DD6.PA4; no longer D6.PA4
- net P53: now also DD6.PA5; no longer D6.PA5
- net P54: now also DD6.PA6; no longer D6.PA6
- net P55: now also DD6.PA7; no longer D6.PA7
- net P56: now also DD6.PB0; no longer D6.PB0
- net P57: now also DD6.PB1; no longer D6.PB1
- net P58: now also DD6.PB2; no longer D6.PB2
- net P59: now also DD6.PB3; no longer D6.PB3
- net P60: now also DD6.PB4; no longer D6.PB4
- net P61: now also DD6.PB5; no longer D6.PB5
- net P62: now also DD6.PB6; no longer D6.PB6
- net P63: now also DD6.PB7; no longer D6.PB7
- net P64: now also DD6.PC0; no longer D6.PC0
- net P65: now also DD6.PC1; no longer D6.PC1
- net P66: now also DD6.PC2; no longer D6.PC2
- net P67: now also DD6.PC3; no longer D6.PC3
- net P68: now also DD6.PC4; no longer D6.PC4
- net P69: now also DD6.PC5; no longer D6.PC5
- net P70: now also DD6.PC6; no longer D6.PC6
- net P71: now also DD6.PC7; no longer D6.PC7
- net P72: now also DD7.PA0; no longer D7.PA0
- net P73: now also DD7.PA1; no longer D7.PA1
- net P74: now also DD7.PA2; no longer D7.PA2
- net P75: now also DD7.PA3; no longer D7.PA3
- net P76: now also DD7.PA4; no longer D7.PA4
- net P77: now also DD7.PA5; no longer D7.PA5
- net P78: now also DD7.PA6; no longer D7.PA6
- net P79: now also DD7.PA7; no longer D7.PA7
- net P80: now also DD7.PB0; no longer D7.PB0
- net P81: now also DD7.PB1; no longer D7.PB1
- net P82: now also DD7.PB2; no longer D7.PB2
- net P83: now also DD7.PB3; no longer D7.PB3
- net P84: now also DD7.PB4; no longer D7.PB4
- net P85: now also DD7.PB5; no longer D7.PB5
- net P86: now also DD7.PB6; no longer D7.PB6
- net P87: now also DD7.PB7; no longer D7.PB7
- net P88: now also DD7.PC0; no longer D7.PC0
- net P89: now also DD7.PC1; no longer D7.PC1
- net P90: now also DD7.PC2; no longer D7.PC2
- net P91: now also DD7.PC3; no longer D7.PC3
- net P92: now also DD7.PC4; no longer D7.PC4
- net P93: now also DD7.PC5; no longer D7.PC5
- net P94: now also DD7.PC6; no longer D7.PC6
- net P95: now also DD7.PC7; no longer D7.PC7
- net R16CS: now also DD24D.I; no longer D24D.I
- net RES: now also DD24E.O, DD6.RESET, DD7.RESET
- net XA0: now also DD29A.1Q, DD6.A0, DD7.A0
- net XA1: now also DD29A.2Q, DD6.A1, DD7.A1
- net XA3: now also DD29A.4Q
- net XA6: now also DD29A.7Q
- net XA7: now also DD29A.8Q

Commit message: .
Parts:
- added R65: 400, rcl:R-EU_R0805
- added R67: 1k, rcl:R-EU_R0805
- added VT1: 315, m_transistor:BJT_NPN_SOT23_BCE
Connections:
- new net N$8: R67.2, VT1.B
- net !IORD: now also R65.2, VT1.E
- net !RDI: now also R67.1
- net +5V: now also DD1P.VCC, DD29P.VCC, DD2P.VCC, VT1.C
- net GND: now also DD1P.GND, DD29P.GND, DD2P.GND, R65.1
Other:
- moved on the sheet: C8, DD1, DD1P, DD2, DD24E, DD29, DD2P, DD4, DD5, DD6, DD7, LPT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

Commit message: .
Parts:
- added DD15, DD16, DD17: К155ЛН3, 74xx-eu:7406N
- added R10, R11: 470, rcl:R-EU_R0805
- added R1A, R1B, R1C, R1D: 2k, rcl:R-EU_R0805
- added VT2: 361g, m_transistor:BJT_PNP_SOT23_BCE
- added VT41: 315, m_transistor:BJT_NPN_SOT23_BCE
- VT1: value 315 -> 361g; device m_transistor:BJT_NPN_SOT23_BCE -> m_transistor:BJT_PNP_SOT23_BCE
Connections:
- new net E1: R10.2, R11.2, VT1.E, VT2.E
- new net N$10: R1B.2, VT1.C
- new net N$11: R10.1, R1A.2, VT1.B
- new net N$12: DD17F.O, R1C.1
- new net N$13: R1D.2, VT2.C
- new net N$14: R11.1, R1C.2, VT2.B
- new net N$9: DD16B.O, R1A.1
- net !IORD: now also VT41.E; no longer VT1.E
- net +5V: now also VT41.C; no longer VT1.C
- net N$8: now also VT41.B; no longer VT1.B
- net P0: now also DD16B.I
- net P1: now also DD17F.I
- net P8: now also DD15A.I
- net P9: now also DD15E.I
- net PA0: now also DD15A.O, R1B.1
- net PA1: now also DD15E.O, R1D.1

Commit message: b0
Parts:
- DD2: value К555КП11 -> К531КП11
Changed lines of the file:
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@@
 <grid distance="0.1" unitdist="inch" unit="inch" style="lines" multiple="1" display="yes" altdistance="0.01" altunitdist="inch" altunit="inch"/>
 <layers>
-<layer number="1" name="Top" color="4" fill="1" visible="yes" active="no"/>
-<layer number="2" name="Route2" color="1" fill="3" visible="yes" active="no"/>
-<layer number="3" name="Route3" color="4" fill="3" visible="yes" active="no"/>
-<layer number="4" name="Route4" color="1" fill="4" visible="yes" active="no"/>
-<layer number="5" name="Route5" color="4" fill="4" visible="yes" active="no"/>
-<layer number="6" name="Route6" color="1" fill="8" visible="yes" active="no"/>
-<layer number="7" name="Route7" color="4" fill="8" visible="yes" active="no"/>
-<layer number="8" name="Route8" color="1" fill="2" visible="yes" active="no"/>
-<layer number="9" name="Route9" color="4" fill="2" visible="yes" active="no"/>
-<layer number="10" name="Route10" color="1" fill="7" visible="yes" active="no"/>
-<layer number="11" name="Route11" color="4" fill="7" visible="yes" active="no"/>
-<layer number="12" name="Route12" color="1" fill="5" visible="yes" active="no"/>
-<layer number="13" name="Route13" color="4" fill="5" visible="yes" active="no"/>
-<layer number="14" name="Route14" color="1" fill="6" visible="yes" active="no"/>
-<layer number="15" name="Route15" color="4" fill="6" visible="yes" active="no"/>
-<layer number="16" name="Bottom" color="1" fill="1" visible="yes" active="no"/>
-<layer number="17" name="Pads" color="2" fill="1" visible="yes" active="no"/>
-<layer number="18" name="Vias" color="2" fill="1" visible="yes" active="no"/>
-<layer number="19" name="Unrouted" color="6" fill="1" visible="yes" active="no"/>
-<layer number="20" name="Dimension" color="15" fill="1" visible="yes" active="no"/>
-<layer number="21" name="tPlace" color="7" fill="1" visible="yes" active="no"/>
-<layer number="22" name="bPlace" color="7" fill="1" visible="yes" active="no"/>
-<layer number="23" name="tOrigins" color="15" fill="1" visible="yes" active="no"/>
-<layer number="24" name="bOrigins" color="15" fill="1" visible="yes" active="no"/>
-<layer number="25" name="tNames" color="7" fill="1" visible="yes" active="no"/>
-<layer number="26" name="bNames" color="7" fill="1" visible="yes" active="no"/>
-<layer number="27" name="tValues" color="7" fill="1" visible="yes" active="no"/>
-<layer number="28" name="bValues" color="7" fill="1" visible="yes" active="no"/>
+<layer number="1" name="Top" color="4" fill="1" visible="no" active="no"/>
+<layer number="2" name="Route2" color="1" fill="3" visible="no" active="no"/>
+<layer number="3" name="Route3" color="4" fill="3" visible="no" active="no"/>
+<layer number="4" name="Route4" color="1" fill="4" visible="no" active="no"/>
+<layer number="5" name="Route5" color="4" fill="4" visible="no" active="no"/>
+<layer number="6" name="Route6" color="1" fill="8" visible="no" active="no"/>
+<layer number="7" name="Route7" color="4" fill="8" visible="no" active="no"/>
+<layer number="8" name="Route8" color="1" fill="2" visible="no" active="no"/>
+<layer number="9" name="Route9" color="4" fill="2" visible="no" active="no"/>
+<layer number="10" name="Route10" color="1" fill="7" visible="no" active="no"/>
+<layer number="11" name="Route11" color="4" fill="7" visible="no" active="no"/>
+<layer number="12" name="Route12" color="1" fill="5" visible="no" active="no"/>
+<layer number="13" name="Route13" color="4" fill="5" visible="no" active="no"/>
+<layer number="14" name="Route14" color="1" fill="6" visible="no" active="no"/>
+<layer number="15" name="Route15" color="4" fill="6" visible="no" active="no"/>
+<layer number="16" name="Bottom" color="1" fill="1" visible="no" active="no"/>
+<layer number="17" name="Pads" color="2" fill="1" visible="no" active="no"/>
+<layer number="18" name="Vias" color="2" fill="1" visible="no" active="no"/>
+<layer number="19" name="Unrouted" color="6" fill="1" visible="no" active="no"/>
+<layer number="20" name="Dimension" color="15" fill="1" visible="no" active="no"/>
+<layer number="21" name="tPlace" color="7" fill="1" visible="no" active="no"/>
+<layer number="22" name="bPlace" color="7" fill="1" visible="no" active="no"/>
+<layer number="23" name="tOrigins" color="15" fill="1" visible="no" active="no"/>
+<layer number="24" name="bOrigins" color="15" fill="1" visible="no" active="no"/>
+<layer number="25" name="tNames" color="7" fill="1" visible="no" active="no"/>
+<layer number="26" name="bNames" color="7" fill="1" visible="no" active="no"/>
+<layer number="27" name="tValues" color="7" fill="1" visible="no" active="no"/>
+<layer number="28" name="bValues" color="7" fill="1" visible="no" active="no"/>
 <layer number="29" name="tStop" color="7" fill="3" visible="no" active="no"/>
 <layer number="30" name="bStop" color="7" fill="6" visible="no" active="no"/>
@@
 <layer number="35" name="tGlue" color="7" fill="4" visible="no" active="no"/>
 <layer number="36" name="bGlue" color="7" fill="5" visible="no" active="no"/>
-<layer number="37" name="tTest" color="7" fill="1" visible="yes" active="no"/>
-<layer number="38" name="bTest" color="7" fill="1" visible="yes" active="no"/>
+<layer number="37" name="tTest" color="7" fill="1" visible="no" active="no"/>
+<layer number="38" name="bTest" color="7" fill="1" visible="no" active="no"/>
 <layer number="39" name="tKeepout" color="4" fill="11" visible="no" active="no"/>
 <layer number="40" name="bKeepout" color="1" fill="11" visible="no" active="no"/>
@@
 <layer number="44" name="Drills" color="7" fill="1" visible="no" active="no"/>
 <layer number="45" name="Holes" color="7" fill="1" visible="no" active="no"/>
-<layer number="46" name="Milling" color="3" fill="1" visible="yes" active="no"/>
-<layer number="47" name="Measures" color="7" fill="1" visible="yes" active="no"/>
-<layer number="48" name="Document" color="7" fill="1" visible="yes" active="no"/>
-<layer number="49" name="Reference" color="7" fill="1" visible="yes" active="no"/>
-<layer number="50" name="dxf" color="7" fill="1" visible="yes" active="no"/>
-<layer number="51" name="tDocu" color="7" fill="1" visible="yes" active="no"/>
-<layer number="52" name="bDocu" color="7" fill="1" visible="yes" active="no"/>
-<layer number="53" name="tGND_GNDA" color="7" fill="1" visible="yes" active="no"/>
-<layer number="54" name="bGND_GNDA" color="7" fill="1" visible="yes" active="no"/>
-<layer number="56" name="wert" color="7" fill="1" visible="yes" active="no"/>
-<layer number="57" name="tCAD" color="7" fill="1" visible="yes" active="no"/>
+<layer number="46" name="Milling" color="3" fill="1" visible="no" active="no"/>
+<layer number="47" name="Measures" color="7" fill="1" visible="no" active="no"/>
+<layer number="48" name="Document" color="7" fill="1" visible="no" active="no"/>
+<layer number="49" name="Reference" color="7" fill="1" visible="no" active="no"/>
+<layer number="50" name="dxf" color="7" fill="1" visible="no" active="no"/>
+<layer number="51" name="tDocu" color="7" fill="1" visible="no" active="no"/>
+<layer number="52" name="bDocu" color="7" fill="1" visible="no" active="no"/>
+<layer number="53" name="tGND_GNDA" color="7" fill="1" visible="no" active="no"/>
+<layer number="54" name="bGND_GNDA" color="7" fill="1" visible="no" active="no"/>
+<layer number="56" name="wert" color="7" fill="1" visible="no" active="no"/>
+<layer number="57" name="tCAD" color="7" fill="1" visible="no" active="no"/>
 <layer number="90" name="Modules" color="7" fill="1" visible="yes" active="yes"/>
 <layer number="91" name="Nets" color="2" fill="1" visible="yes" active="yes"/>
@@
 <part name="DD1" library="74xx-eu" deviceset="74*245" device="N" technology="LS" value="К555АП6"/>
 <part name="P+9" library="supply1v" deviceset="+5V" device=""/>
-<part name="DD2" library="74xx-eu" deviceset="74*257" device="N" technology="S" value="К555КП11"/>
+<part name="DD2" library="74xx-eu" deviceset="74*257" device="N" technology="S" value="К531КП11"/>
 <part name="GND14" library="supply1v" deviceset="GND" device=""/>
 <part name="DD29" library="74xx-eu" deviceset="74*374" device="N" technology="LS" value="К555ИР23"/>

Commit message: d1
Parts:
- added R1: 3k3, rcl:R-EU_M0805
- added R38: 1k, rcl:R-EU_M0805
- added R50: 510, rcl:R-EU_M0805
- added R54: 100, rcl:R-EU_M0805
- added VT29: КТ972, m_transistor:BJT_NPN_TO126_V_ECB
- added VT33: КТ805, m_transistor:BJT_NPN_TO220_V_ECB
- added VT37: КТ973, m_transistor:BJT_PNP_TO126_V_ECB
- added X2: (no value), Разъёмы штырьковые 2.54мм:PINHD-2X20
Connections:
- new net N$15: DA12A.-IN, R1.1, R38.2
- new net N$16: R50.2, R54.2, VT29.E, VT33.B
- new net N$19: R46.2, R50.1, VT29.B, VT37.B
- net +27V: now also VT29.C, VT33.C
- net -5V: now also VT37.C
- net E1: now also R1.2, R54.1, VT33.E, VT37.E
- net GND: now also R38.1
- net P67: no longer DD8.BIT2
- net P68: now also DD8.BIT2
- net P84: no longer DD10.BIT1
- net P85: now also DD10.BIT1

Commit message: .
Parts:
- added C7: 390, rcl:C-EUC0805
- added DA1: КР574УД2А, ОУ:КР574УД2А
- added R2, R3, R4, R5, R6, R7: (no value), rcl:R-EU_M0805
- added R8, R9: 1k6, rcl:R-EU_M0805
- added VT10, VT11, VT12, VT13, VT3, VT5, VT9: BJT_NPN_TO126_V_ECB, m_transistor:BJT_NPN_TO126_V_ECB
- added VT4, VT6, VT7, VT8: BJT_PNP_TO126_V_ECB, m_transistor:BJT_PNP_TO126_V_ECB
Connections:
- new net N$17: VT3.B, VT4.B
- new net N$18: R3.1
- new net N$20: VT3.C, VT4.C, VT5.B, VT6.C, VT7.B
- new net N$22: VT11.B, VT5.C, VT6.B, VT7.C, VT8.B, VT9.B
- new net N$23: R4.1
- new net N$24: VT10.B, VT8.C, VT9.C
- new net N$26: R3.2, R5.2, R6.1
- new net N$27: R2.1, VT10.C, VT11.C
- new net N$28: R4.2, R6.2, R7.1
- new net N$32: R9.1, VT12.B
- new net N$33: C7.1, VT13.C
- new net N$34: R8.1, VT13.B
- new net N$36: C7.2, DA1A.+IN, R2.2, R5.1, VT12.C
- net +14V: now also VT4.E, VT6.E, VT7.E, VT8.E
- net +5V: now also R8.2, R9.2
- net +7V: now also VT11.E
- net GND: now also R7.2, VT10.E, VT12.E, VT13.E, VT3.E, VT5.E, VT9.E
Other:
- note added: "1"
- note added: "14"
- note added: "15"
- note added: "2"
- note added: "3"
- note added: "4"
