File: uniprog21.sch (EAGLE design)
At the start: 91 parts

Commit message: .
Parts:
- removed C1, C2, C7: 390, rcl:C-EUC0805
- removed DA1: КР574УД2А, ОУ:КР574УД2А
- removed DP10: i8748/9, ic-package:DIL40
- removed DP4: 556РТ5-7,16, ic-package:DIL24-6
- removed DP8: 2x64-2x512, ic-package:DIL28
- removed DP9: 2716-2732, ic-package:DIL24-6
- removed LPT: (no value), con-subd:M25HP
- removed R1: 3k3, rcl:R-EU_M0805
- removed R2, R3, R4, R5, R6, R7: (no value), rcl:R-EU_M0805
- removed R38: 1k, rcl:R-EU_M0805
- removed R46, R47: 270, rcl:R-EU_M0805
- removed R50: 510, rcl:R-EU_M0805
- removed R54: 100, rcl:R-EU_M0805
- removed R8, R9: 1k6, rcl:R-EU_M0805
- removed VT10, VT11, VT12, VT13, VT3, VT5, VT9: BJT_NPN_TO126_V_ECB, m_transistor:BJT_NPN_TO126_V_ECB
- removed VT29: КТ972, m_transistor:BJT_NPN_TO126_V_ECB
- removed VT33: КТ805, m_transistor:BJT_NPN_TO220_V_ECB
- removed VT37: КТ973, m_transistor:BJT_PNP_TO126_V_ECB
- removed VT4, VT6, VT7, VT8: BJT_PNP_TO126_V_ECB, m_transistor:BJT_PNP_TO126_V_ECB
- added C1N, C2N: 390, rcl:C-EUC0805
- added CX2, CX49: 100n, rcl:C-EUC0805
- added DP10U: i8748/9, ic-package:DIL40
- added DP11N: 556РТ5, ic-package:DIL24-6
- added DP4U/N(11): 556РТ5,6,7,16/6,7,16, ic-package:DIL24-6
- added DP8U/DP9N: 2x64-2x512, ic-package:DIL28
- added DP9U/DP10N: 2716-2732, ic-package:DIL24-6
- added LPT26PINS: (no value), Разъёмы штырьковые 2.54мм:PINHD-2X13
- added LPTDB25_: (no value), con-subd:M25HP
- added R1/R87N, R92N: 3k3, rcl:R-EU_M0805
- added R38/R88N, R93N: 1k, rcl:R-EU_M0805
- added R46/R89N, R94N: 270, rcl:R-EU_M0805
- added R50/R90N, R95N: 510, rcl:R-EU_M0805
- added R54/R91N, R96N: 100, rcl:R-EU_M0805
- added VT29N, VT30N: КТ972, m_transistor:BJT_NPN_TO126_V_ECB
- added VT33N, VT34N: КТ805, m_transistor:BJT_NPN_TO220_V_ECB
- added VT37N, VT38N: КТ973, m_transistor:BJT_PNP_TO126_V_ECB
- added X1: (no value), Разъёмы штырьковые 2.54мм:PINHD-2X20
- DP2U/N: value 556РТ12-15 -> 556РТ12,13,14,15
- DP3U/N: value 556РТ4 -> 556РТ4,11
- renumbered DP1 to DP1U/N, DP11 to DP11U/DP12N, DP2 to DP2U/N, DP3 to DP3U/N, DP5 to DP5U/N, DP6 to DP6U/N, DP7 to DP7U/DP8N
Connections:
- removed net N$17: VT3.B, VT4.B
- removed net N$18: R3.1
- removed net N$2: C2.1, DD26C.O
- removed net N$27: R2.1, VT10.C, VT11.C
- removed net N$28: R4.2, R6.2, R7.1
- removed net N$32: R9.1, VT12.B
- removed net N$33: C7.1, VT13.C
- removed net N$34: R8.1, VT13.B
- removed net N$36: C7.2, DA1A.+IN, R2.2, R5.1, VT12.C
- removed net N$7: DA12B.OUT, R47.1
- new net N$21: DD10.VDD, DD11.VDD
- new net N$25: R95N.2, R96N.2, VT30N.E, VT34N.B
- net !ADWR: now also LPT26PINS.2; no longer LPT.14
- net !EN1: now also C1N.2; no longer C1.2
- net !EN2: now also C2N.2; no longer C2.2
- net !EN3: now also DD27F.O; no longer DD26F.O
- net !IOWR: now also LPT26PINS.8; no longer LPT.17
- net !RDI: now also LPT26PINS.6; no longer LPT.16
- net +14V: no longer DD10.VDD, DD11.VDD, VT4.E, VT6.E, VT7.E, VT8.E
- net +27V: now also CX2.1, CX49.1, VT29N.C, VT30N.C, VT33N.C, VT34N.C; no longer VT29.C, VT33.C
- net +5V: now also DD26P.VCC; no longer R8.2, R9.2
- net +7V: no longer DD10.OUT1, DD11.OUT1, VT11.E
- net -5V: now also CX2.2, CX49.2, VT37N.C, VT38N.C; no longer VT37.C
- net E1: now also R1/R87N.2, R54/R91N.1, VT33N.E, VT37N.E; no longer R1.2, R54.1, VT33.E, VT37.E
- net E2: now also R92N.2, R96N.1, VT34N.E, VT38N.E
- net GND: now also DD26P.GND, LPT26PINS.10, LPT26PINS.12, LPT26PINS.14, LPT26PINS.16, LPT26PINS.18, LPT26PINS.20, LPT26PINS.22, LPT26PINS.24, LPT26PINS.26, R38/R88N.1, R93N.1; no longer LPT.19, LPT.20, LPT.21, LPT.22, LPT.23, LPT.24, LPT.25, R38.1, R7.2, VT10.E, VT12.E, VT13.E, VT3.E, VT5.E, VT9.E
- net N$1: now also C1N.1; no longer C1.1
- net N$15: now also R1/R87N.1, R38/R88N.2; no longer R1.1, R38.2
- net N$16: now also R50/R90N.2, R54/R91N.2, VT29N.E, VT33N.B; no longer R50.2, R54.2, VT29.E, VT33.B
- net N$19: now also R46/R89N.2, R50/R90N.1, VT29N.B, VT37N.B; no longer R46.2, R50.1, VT29.B, VT37.B
- net N$20: now also DD10.OUT1, DD11.OUT1; no longer VT3.C, VT4.C, VT5.B, VT6.C, VT7.B
- net N$22: now also C2N.1, DD26C.O; no longer VT11.B, VT5.C, VT6.B, VT7.C, VT8.B, VT9.B
- net N$23: now also DA12B.OUT, R94N.1; no longer R4.1
- net N$24: now also DA12B.-IN, R92N.1, R93N.2; no longer VT10.B, VT8.C, VT9.C
- net N$26: now also R94N.2, R95N.1, VT30N.B, VT38N.B; no longer R3.2, R5.2, R6.1
- net N$3: now also DD27E.O; no longer DD26E.O
- net N$6: now also R46/R89N.1; no longer R46.1
- net P86: now also DD27E.I; no longer DD26E.I
- net P87: now also DD27F.I; no longer DD26F.I
- net PA13: now also DP10U.36
- net PA14: now also DP10U.37
- net PA15: now also DP10U.38; no longer DP10.38
- net XD0: now also LPT26PINS.3; no longer LPT.2
- net XD1: now also LPT26PINS.5; no longer LPT.3
- net XD2: now also LPT26PINS.7; no longer LPT.4
- net XD3: now also LPT26PINS.9; no longer LPT.5
- net XD4: now also LPT26PINS.11; no longer LPT.6
- net XD5: now also LPT26PINS.13; no longer LPT.7
- net XD6: now also LPT26PINS.15; no longer LPT.8
- net XD7: now also LPT26PINS.17; no longer LPT.9
- net XI0: now also LPT26PINS.25; no longer LPT.13
- net XI1: now also LPT26PINS.23; no longer LPT.12
- net XI2: now also LPT26PINS.19; no longer LPT.10
- net XI3: now also LPT26PINS.21; no longer LPT.11
- net XI4: now also LPT26PINS.1; no longer LPT.1
Other:
- note added: "DA12P"
- note added: "DA13P"
- note added: "КМ1816ВЕ48"
- note added: "КМ1830ВЕ751"
- note added: "РТ5 pin22 E4 РТ16 pin22 E3"
- note removed: "1"
- note removed: "14"
- note removed: "15"
- note removed: "2"
- note removed: "3"
- note removed: "4"
- note removed: "D12P"
- note removed: "D13P"
