File: uniprog21.sch (EAGLE design)
At the start: 82 parts

Commit message: .
Parts:
- removed C3, C4: 390, rcl:C-EUC0805
- added C3N, C4N: 390, rcl:C-EUC0805
- added R100N, R105N: 510, rcl:R-EU_M0805
- added R101, R106N: 100, rcl:R-EU_M0805
- added R102N, R97N: 3k3, rcl:R-EU_M0805
- added R103N, R98N: 1k, rcl:R-EU_M0805
- added R104N, R99N: 270, rcl:R-EU_M0805
- added VT31N, VT32N: КТ972, m_transistor:BJT_NPN_TO126_V_ECB
- added VT35N, VT36N: КТ805, m_transistor:BJT_NPN_TO220_V_ECB
- added VT39N, VT40N: КТ973, m_transistor:BJT_PNP_TO126_V_ECB
Connections:
- removed net N$20: DD10.OUT1, DD11.OUT1
- removed net N$21: DD10.VDD, DD11.VDD
- removed net N$3: C3.1, DD27E.O
- removed net N$4: C4.1, DD27A.O
- new net N$17: DA13A.-IN, R97N.1, R98N.2
- new net N$18: R100N.2, R101.2, VT31N.E, VT35N.B
- new net N$2: C3N.1, DD27E.O
- new net N$27: R100N.1, R99N.2, VT31N.B, VT39N.B
- new net N$28: C4N.1, DD27A.O
- new net N$29: DA13B.OUT, R104N.1
- new net N$30: DA13B.-IN, R102N.1, R103N.2
- new net N$31: R105N.2, R106N.2, VT32N.E, VT36N.B
- new net N$32: R104N.2, R105N.1, VT32N.B, VT40N.B
- new net N$7: DA13A.OUT, R99N.1
- net !EN3: now also C3N.2, DA13A.+IN; no longer C3.2
- net !EN4: now also C4N.2, DA13B.+IN; no longer C4.2
- net +14V: now also DD10.VDD, DD11.VDD
- net +27V: now also VT31N.C, VT32N.C, VT35N.C, VT36N.C
- net +5V: now also DD27P.VCC
- net +7V: now also DD10.OUT1, DD11.OUT1
- net -5V: now also VT39N.C, VT40N.C
- net E3: now also R101.1, R97N.2, VT35N.E, VT39N.E
- net E4: now also R102N.2, R106N.1, VT36N.E, VT40N.E
- net GND: now also DD27P.GND, R103N.1, R98N.1
