File: uniprog21.sch (EAGLE design)
At the start: 98 parts

Commit message: .
Parts:
- removed R10, R11: 470, rcl:R-EU_R0805
- removed R1A, R1B, R1C, R1D: 2k, rcl:R-EU_R0805
- removed R5A, R5B, R5C, R5D, R5E, R5F, R5G, R5H: 1k, rcl:R-EU_M0805
- added JP1: (no value), Разъёмы штырьковые 2.54мм:PINHD-1X6
- added JP2: (no value), Разъёмы штырьковые 2.54мм:PINHD-1X4
- added JP3: (no value), Разъёмы штырьковые 2.54мм:PINHD-1X11
- added JP5: (no value), Разъёмы штырьковые 2.54мм:PINHD-1X5
- added R83(R62U2.1), R84(R5U2.1), R85(R6U2.1), R86(R8U2.1): 1k, resistor-sil:G09R
- added RN1: НР-1-1-1-8 470 5%, resistor-dil:8R-N
- added RN10: НР-1-1-1-8 2k, resistor-dil:8R-N
- added VD1, VD10, VD11, VD12, VD13, VD14, VD15, VD16, VD2, VD3, VD4, VD5, VD6, VD7, VD8, VD9: КД522, diode:1N4148DO35-7
- VT1, VT2: value 361g -> КТ361Г; device m_transistor:BJT_PNP_SOT23_BCE -> m_transistor:BJT_PNP_TO-92_ECB
Connections:
- new net N$20: VD9.A
- new net N$21: R85(R6U2.1).3, VD10.C
- new net N$3: R85(R6U2.1).2, VD9.C
- new net N$33: R85(R6U2.1).4, VD11.C
- new net N$34: R85(R6U2.1).5, VD12.C
- new net N$35: R85(R6U2.1).6, VD13.C
- new net N$36: R85(R6U2.1).7, VD14.C
- new net N$37: R85(R6U2.1).8, VD15.C
- new net N$38: R85(R6U2.1).9, VD16.C
- new net N$4: VD10.A
- net !IOWR: now also JP1.2
- net +5V: now also R83(R62U2.1).1, R84(R5U2.1).1; no longer R5A.2, R5B.2, R5C.2, R5D.2, R5E.2, R5F.2, R5G.2, R5H.2
- net E1: now also RN1A.2, RN1C.2; no longer R10.2, R11.2
- net N$10: now also RN1B.2; no longer R1B.2
- net N$11: now also RN10A.2, RN1A.1; no longer R10.1, R1A.2
- net N$12: now also RN10B.1; no longer R1C.1
- net N$13: now also RN1D.2; no longer R1D.2
- net N$14: now also RN10B.2, RN1C.1; no longer R11.1, R1C.2
- net N$9: now also RN10A.1; no longer R1A.1
- net P72: now also JP2.4
- net P73: now also JP2.3
- net P74: now also JP2.2
- net P75: now also JP2.1
- net P76: now also JP1.6
- net P77: now also JP1.5
- net P78: now also JP1.4
- net P79: now also JP1.3
- net P80: now also JP3.9
- net P81: now also JP3.10
- net P82: now also JP3.11
- net P83: now also JP5.1
- net P84: now also JP5.2
- net P85: now also JP5.3
- net P86: now also JP5.4
- net P87: now also JP5.5
- net P88: now also JP3.5
- net P89: now also JP3.6
- net P90: now also JP3.7
- net P91: now also JP3.8
- net P92: now also JP3.4
- net P93: now also JP3.3
- net P94: now also JP3.2
- net P95: now also JP3.1
- net PA0: now also RN1B.1; no longer R1B.1
- net PA1: now also RN1D.1; no longer R1D.1
- net PD10: now also R84(R5U2.1).4; no longer R5C.1
- net PD11: now also R84(R5U2.1).5, R84(R5U2.1).6; no longer R5D.1, R5E.1
- net PD13: now also R84(R5U2.1).7; no longer R5F.1
- net PD14: now also R84(R5U2.1).8; no longer R5G.1
- net PD15: now also R84(R5U2.1).9; no longer R5H.1
- net PD8: now also R84(R5U2.1).2; no longer R5A.1
- net PD9: now also R84(R5U2.1).3; no longer R5B.1
- net RES: now also JP1.1
Other:
- note added: "NOTE =16 E1-E4 =4 +5 +7 +14 GND =4 ==24"
- note added: "NOTE P64-P69P70-71 P72-P77 78-79 95 =32 E1-E4 x2 =8 ==40 +5 +7 +14 GND =4 ==44"
- note added: "NOTE на 1 элемент 6 вход вв55 D7(КР580ВВ55А) P72-P95 ==32 вход !EN! 1шт. итого 7 входов"

Commit message: .
Parts:
- removed DD16: К155ЛН3, 74xx-eu:7406N
- added (DD16.1)DD14, D-0, D-1, D-2: К155ЛН3, 74xx-eu:7406N
- added D1, D10, D11, D2, D3, D4, D5, D6, D7, D8, D9: Д310, diode:1N5060GP
- added R1, R10, R11, R12, R19, R2, R20, R21, R3: 2k, rcl:R-EU_R0805
- added R13, R14, R15, R16, R17, R18, R22, R23, R24, R25, R26, R27, R4, R5, R6, R7, R8, R9: 470, rcl:R-EU_R0805
- added VT10, VT11, VT3, VT4, VT5, VT6, VT7, VT8, VT9: КТ361Г, m_transistor:BJT_PNP_TO-92_ECB
- R1/R87N, R100N, R101, R102N, R103N, R104N, R105N, R106N, R38/R88N, R46/R89N, R50/R90N, R54/R91N, R92N, R93N, R94N, R95N, R96N, R97N, R98N, R99N: device rcl:R-EU_M0805 -> rcl:R-EU_R0805
- renumbered DD15 to (DD15.1)DD15, JP1 to P_DAC4, JP2 to P_DAC1, JP3 to P_DAC2, JP5 to P_DAC3
Connections:
- new net N$39: D1.A, RN1B.1
- new net N$40: D2.A, RN1D.1
- new net N$41: R1.2, R4.1, VT3.B
- new net N$42: D6.A, VT3.C
- new net N$43: D6.C, R5.2
- new net N$44: D-0A.O, R1.1
- new net N$45: R2.2, R6.1, VT4.B
- new net N$46: D3.A, VT4.C
- new net N$47: D-0F.O, R5.1
- new net N$48: R3.2, R8.1, VT5.B
- new net N$49: D4.A, VT5.C
- new net N$50: D-0D.O, R9.1
- new net N$51: D-0C.O, R3.1
- new net N$52: D-0B.O, R2.1
- new net N$53: D4.C, R9.2
- new net N$54: D3.C, R7.2
- new net N$55: D-0E.O, R7.1
- new net N$56: R10.2, R13.1, VT7.B
- new net N$57: D5.A, VT7.C
- new net N$58: D-1A.O, R10.1
- new net N$59: R11.2, R15.1, VT8.B
- new net N$60: D7.A, VT8.C
- new net N$61: R12.2, R17.1, VT9.B
- new net N$62: D8.A, VT9.C
- new net N$63: D-1C.O, R12.1
- new net N$64: D-1B.O, R11.1
- new net N$65: D5.C, R14.2
- new net N$66: D-1F.O, R14.1
- new net N$67: D-1D.O, R18.1
- new net N$68: D8.C, R18.2
- new net N$69: D7.C, R16.2
- new net N$70: D-1E.O, R16.1
- new net N$71: R19.2, R22.1, VT6.B
- new net N$72: D9.A, VT6.C
- new net N$73: D-2A.O, R19.1
- new net N$74: R20.2, R24.1, VT10.B
- new net N$75: D10.A, VT10.C
- new net N$76: R21.2, R26.1, VT11.B
- new net N$77: D11.A, VT11.C
- new net N$78: D-2C.O, R21.1
- new net N$79: D-2B.O, R20.1
- new net N$80: D9.C, R23.2
- new net N$81: D-2F.O, R23.1
- new net N$82: D-2D.O, R27.1
- new net N$83: D11.C, R27.2
- new net N$84: D10.C, R25.2
- new net N$85: D-2E.O, R25.1
- net E1: now also R13.2, R15.2, R17.2, R22.2, R24.2, R26.2, R4.2, R6.2, R8.2, VT10.E, VT11.E, VT3.E, VT4.E, VT5.E, VT6.E, VT7.E, VT8.E, VT9.E
- net N$9: now also (DD16.1)DD14C.O; no longer DD16B.O
- net P0: now also (DD16.1)DD14C.I; no longer DD16B.I
- net PA0: now also D1.C; no longer RN1B.1
- net PA1: now also D2.C; no longer RN1D.1
Other:
- moved on the sheet: RN1B, RN1D
